Commit message: init

File: urdf/arm5.urdf (robot description, URDF)
Before this commit: robot arm5, 6 links, 5 joints
Links:
- added link virtual_base_link
- link Empty_Link1: mass 0.060372 -> 0.0603720269298029
- link Empty_Link2: mass 0.36978 -> 0.369779302354558
- link Empty_Link3: mass 0.16255 -> 0.162548001883722
- link Empty_Link4: mass 0.10047 -> 0.100466627587425
- link Empty_Link5: mass 0.038021 -> 0.0380214590684831
- link base_link: mass 6.5373 -> 6.53725957238719
Joints:
- added joint base_joint: type fixed, parent virtual_base_link, child base_link
- joint j1: axis 0 0 1 -> 0 0 -1; origin xyz=-0.1255 0 0 rpy=-1.5708 1.5315 1.5708 -> xyz=0.1255 0 0 rpy=-1.5708 1.5315 -1.5708
- joint j2: axis 0 0 1 -> 0 0 -1; limit lower=-1.5708 upper=1.5708 effort=0 velocity=0 -> lower=-1.57 upper=1.57 effort=0 velocity=0
- joint j3: axis 0 0 1 -> 0 0 -1
- joint j5: axis 0 0 1 -> 0 0 -1; limit lower=-1.5708 upper=1.5708 effort=0 velocity=0 -> lower=-1.57 upper=1.57 effort=0 velocity=0
